Commit message: switched to python. To manuver around c++ implementation issues for now. (will have to solve later)

File: src/mark_ii_moveit_new/config/MarkII_urdf.ros2_control.xacro (robot description, xacro)
@@ -1,17 +1,6 @@
 <robot xmlns:xacro="http://ros.org/wiki/xacro">
-    <xacro:arg name="use_real_hardware" default="true" />
-    <xacro:unless value="$(arg use_real_hardware)">
-        <xacro:property name="initial_positions" value="${dict(
-            'base_link_Revolute-1': 0.0,
-            'link1_Revolute-3': 0.0,
-            'link2_Revolute-4': 0.0,
-            'link3_Revolute-5': 0.0,
-            'link4_Revolute-6': 0.0,
-            'link5_Revolute-7': 0.0,
-            'link6_Slider-8': 0.0
-        )}" />
-    </xacro:unless>
-    <ros2_control name="MarkIIHardware" type="system">
-        <xacro:if value="$(arg use_real_hardware)">
+    <xacro:macro name="arm_description_ros2_control" params="name initial_positions_file">
+        <xacro:property name="initial_positions" value="${load_yaml(initial_positions_file)['initial_positions']}"/>
+        <ros2_control name="MarkIIHardware" type="system">
             <hardware>
                 <plugin>simple_arm/ArmHardware</plugin>
@@ -19,67 +8,55 @@
                 <param name="baudrate">1000000</param>
             </hardware>
-        </xacro:if>
-        <xacro:unless value="$(arg use_real_hardware)">
-            <hardware>
-                <plugin>mock_components/GenericSystem</plugin>
-            </hardware>
-        </xacro:unless>
-        <!-- Joint Interfaces -->
-        <joint name="base_link_Revolute-1">
-            <command_interface name="position" />
-            <state_interface name="position">
-                <xacro:unless value="$(arg use_real_hardware)">
+            <!-- Joint Interfaces -->
+            <joint name="base_link_Revolute-1">
+                <command_interface name="position" />
+                <state_interface name="position">
                     <param name="initial_value">${initial_positions['base_link_Revolute-1']}</param>
-                </xacro:unless>
-            </state_interface>
-        </joint>
-        <joint name="link1_Revolute-3">
-            <command_interface name="position" />
-            <state_interface name="position">
-                <xacro:unless value="$(arg use_real_hardware)">
+                </state_interface>
+                <state_interface name="velocity"/>
+            </joint>
+            <joint name="link1_Revolute-3">
+                <command_interface name="position" />
+                <state_interface name="position">
                     <param name="initial_value">${initial_positions['link1_Revolute-3']}</param>
-                </xacro:unless>
-            </state_interface>
-        </joint>
-        <joint name="link2_Revolute-4">
-            <command_interface name="position" />
-            <state_interface name="position">
-                <xacro:unless value="$(arg use_real_hardware)">
+                </state_interface>
+                <state_interface name="velocity"/>
+            </joint>
+            <joint name="link2_Revolute-4">
+                <command_interface name="position" />
+                <state_interface name="position">
                     <param name="initial_value">${initial_positions['link2_Revolute-4']}</param>
-                </xacro:unless>
-            </state_interface>
-        </joint>
-        <joint name="link3_Revolute-5">
-            <command_interface name="position" />
-            <state_interface name="position">
-                <xacro:unless value="$(arg use_real_hardware)">
+                </state_interface>
+                <state_interface name="velocity"/>
+            </joint>
+            <joint name="link3_Revolute-5">
+                <command_interface name="position" />
+                <state_interface name="position">
                     <param name="initial_value">${initial_positions['link3_Revolute-5']}</param>
-                </xacro:unless>
-            </state_interface>
-        </joint>
-        <joint name="link4_Revolute-6">
-            <command_interface name="position" />
-            <state_interface name="position">
-                <xacro:unless value="$(arg use_real_hardware)">
+                </state_interface>
+                <state_interface name="velocity"/>
+            </joint>
+            <joint name="link4_Revolute-6">
+                <command_interface name="position" />
+                <state_interface name="position">
                     <param name="initial_value">${initial_positions['link4_Revolute-6']}</param>
-                </xacro:unless>
-            </state_interface>
-        </joint>
-        <joint name="link5_Revolute-7">
-            <command_interface name="position" />
-            <state_interface name="position">
-                <xacro:unless value="$(arg use_real_hardware)">
+                </state_interface>
+                <state_interface name="velocity"/>
+            </joint>
+            <joint name="link5_Revolute-7">
+                <command_interface name="position" />
+                <state_interface name="position">
                     <param name="initial_value">${initial_positions['link5_Revolute-7']}</param>
-                </xacro:unless>
-            </state_interface>
-        </joint>
-        <joint name="link6_Slider-8">
-            <command_interface name="position" />
-            <state_interface name="position">
-                <xacro:unless value="$(arg use_real_hardware)">
+                </state_interface>
+                <state_interface name="velocity"/>
+            </joint>
+            <joint name="link6_Slider-8">
+                <command_interface name="position" />
+                <state_interface name="position">
                     <param name="initial_value">${initial_positions['link6_Slider-8']}</param>
-                </xacro:unless>
-            </state_interface>
-        </joint>
-    </ros2_control>
+                </state_interface>
+                <state_interface name="velocity"/>
+            </joint>
+        </ros2_control>
+    </xacro:macro>
 </robot>

File: src/mark_ii_moveit_new/config/MarkII_urdf.urdf.xacro (robot description, xacro)
@@ -1,10 +1,5 @@
+<?xml version="1.0"?>
 <robot name="MarkII_urdf" xmlns:xacro="http://ros.org/wiki/xacro">
     <xacro:include filename="$(find simple_arm)/description/MarkII_urdf.urdf" />
     <xacro:include filename="$(find mark_ii_moveit_new)/config/MarkII_urdf.ros2_control.xacro" />
-    <link name="world" />
-    <joint name="world_joint" type="fixed">
-        <origin rpy="0 0 0" xyz="0 0 0" />
-        <parent link="world" />
-        <child link="base_link" />
-    </joint>
 </robot>

File: src/simple_arm/description/MarkII_urdf.urdf (robot description, URDF)
Before this commit: robot MarkII_urdf, 10 links, 9 joints
Links:
- removed link gripper_ee
- added link gripper
- link base_link: mass 0.39602545916549503 -> None
Joints:
- removed joint link6_to_gripper_ee
- added joint link6_to_gripper: type fixed, parent link6, child gripper, origin xyz=0 0 0.05 rpy=0 0 0
