Commit message: still no solution found will keep looking and trying

File: src/simple_arm/description/MarkII_urdf.urdf (robot description, URDF)
Before this commit: robot MarkII_urdf, 10 links, 9 joints
Joints:
- joint link1_Revolute-3: limit lower=-0.349066 upper=3.490659 effort=1000000.0 velocity=1000000.0 -> lower=-3.490659 upper=0.349066 effort=1000000.0 velocity=1000000.0

Commit message: only little progress

File: src/simple_arm/description/MarkII_urdf.urdf (robot description, URDF)
Before this commit: robot MarkII_urdf, 10 links, 9 joints
Joints:
- joint base_link_Revolute-1: axis 0.0 -5.319298016155975e-16 1.0 -> 0.0 0.0 1.0
- joint link1_Revolute-3: axis -1 -9.86076131526265e-32 -2.91433543964095e-15 -> -1 0.0 0.0
- joint link2_Revolute-4: axis -0.9999999999999999 -9.860761315262648e-32 -3.1554436208840472e-30 -> -1 0.0 0.0
- joint link3_Revolute-5: axis 0.0 1.0 -3.6755994903979264e-17 -> 0.0 1.0 0.0
- joint link4_Revolute-6: axis 1.0 0.0 1.6307655579902438e-16 -> 1.0 0.0 0.0
- joint link5_Revolute-7: axis 0.0 1.0 -4.3859902218644406e-16 -> 0.0 1.0 0.0
- joint link6_Slider-8: axis 1.0040277787914188e-14 1.3663471679475653e-30 0.9999999999999999 -> 0.0 0.0 1.0
- joint link7_Slider-9: axis 0 0 1 -> 0.0 0.0 1.0
